File: Charger/Charger Junction PCB V1.01/Junction PCB.kicad_sch (KiCad schematic)
At the start: 8 parts, among them J3 Charger CAN, J4 Tractive Battery, J5 12V Battery, SW1 J1772 Dummy Enable (BMS Overr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

Commit message: TVS diode PN added
Parts:
- added J6: Charger, symbol Connector:Conn_01x06_Socket
- added J7: E-Stop, symbol Connector:Conn_01x02_Socket
- D1: value SMAJ12CA -> Comchip ATV02W120B-HF
- D2: footprint Diode_THT:D_DO-35_SOD27_P7.62mm_Horizontal -> Diode_SMD:D_SOD-123
- J3: value Charger CAN -> J1772 In
Connections:
- net control_pilot_in: now also J3.1 (Pin_1)
- net control_proximity: now also J3.2 (Pin_2)
Changed lines of the file:
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@@
+		)
+	)
+	(hierarchical_label "control_proximity"
+		(shape input)
+		(at 111.76 121.92 90)
+		(effects
+			(font
+				(size 1.27 1.27)
+			)
+			(justify left)
+		)
+	)
+	(hierarchical_label "control_pilot_in"
+		(shape input)
+		(at 114.3 121.92 90)
+		(effects
+			(font
+				(size 1.27 1.27)
+			)
+			(justify left)
 		)
 	)
@@
 		)
 		(instances
-			(project "Charger Master"
+			(project "Charger Junction PCB V1.01"
 				(path "/75f6fa4d-fba8-4d29-9299-863888d8bb95/37a81acb-7a57-4259-903f-870230a418d1/a56e1ce8-18bc-4320-87c8-0a13c817c3cf"
 					(reference "J4")
@@
 		)
 		(instances
-			(project "Charger Master"
+			(project "Charger Junction PCB V1.01"
 				(path "/75f6fa4d-fba8-4d29-9299-863888d8bb95/37a81acb-7a57-4259-903f-870230a418d1/a56e1ce8-18bc-4320-87c8-0a13c817c3cf"
 					(reference "R1")
+					(unit 1)
+				)
+			)
+		)
+	)
+	(symbol
+		(lib_id "Connector:Conn_01x02_Socket")
+		(at 236.22 127 270)
+		(unit 1)
+		(body_style 1)
+		(exclude_from_sim no)
+		(in_bom yes)
+		(on_board yes)
+		(in_pos_files yes)
+		(dnp no)
+		(fields_autoplaced yes)
+		(property "Reference" "J7"
+			(at 237.49 125.0949 90)
+			(show_name no)
+			(do_not_autoplace no)
+			(effects
+				(font
+					(size 1.27 1.27)
+				)
+				(justify left)
+			)
+		)
+		(property "Value" "E-Stop"
+			(at 237.49 127.6349 90)
+			(show_name no)
+			(do_not_autoplace no)
+			(effects
+				(font
+					(size 1.27 1.27)
+				)
+				(justify left)
+			)
+		)
+		(property "Footprint" ""
+			(at 236.22 127 0)
+			(hide yes)
+			(show_name no)
+			(do_not_autoplace no)
+			(effects
+				(font
+					(size 1.27 1.27)
+				)
+			)
+		)
+		(property "Datasheet" ""
+			(at 236.22 127 0)
+			(hide yes)
+			(show_name no)
+			(do_not_autoplace no)
+			(effects
+				(font
+					(size 1.27 1.27)
+				)
+			)
+		)
+		(property "Description" "Generic connector, single row, 01x02, script generated"
+			(at 236.22 127 0)
+			(hide yes)
+			(show_name no)
+			(do_not_autoplace no)
+			(effects
+				(font
+					(size 1.27 1.27)
+				)
+			)
+		)
+		(pin "1"
+		)
+		(pin "2"
+		)
+		(instances
+			(project "Charger Junction PCB V1.01"
+				(path "/75f6fa4d-fba8-4d29-9299-863888d8bb95/37a81acb-7a57-4259-903f-870230a418d1/a56e1ce8-18bc-4320-87c8-0a13c817c3cf"
+					(reference "J7")
 					(unit 1)
 				)
@@
 		)
 		(instances
-			(project "Charger Master"
+			(project "Charger Junction PCB V1.01"
 				(path "/75f6fa4d-fba8-4d29-9299-863888d8bb95/37a81acb-7a57-4259-903f-870230a418d1/a56e1ce8-18bc-4320-87c8-0a13c817c3cf"
 					(reference "#PWR02")
@@
 		)
 		(instances
-			(project "Charger Master"
+			(project "Charger Junction PCB V1.01"
 				(path "/75f6fa4d-fba8-4d29-9299-863888d8bb95/37a81acb-7a57-4259-903f-870230a418d1/a56e1ce8-18bc-4320-87c8-0a13c817c3cf"
 					(reference "#PWR03")
@@
 	)
 	(symbol
+		(lib_id "Connector:Conn_01x06_Socket")
+		(at 148.59 127 270)
+		(unit 1)
+		(body_style 1)
+		(exclude_from_sim no)
+		(in_bom yes)
+		(on_board yes)
+		(in_pos_files yes)
+		(dnp no)
+		(fields_autoplaced yes)
+		(property "Reference" "J6"
+			(at 147.32 129.54 90)
+			(show_name no)
+			(do_not_autoplace no)
+			(effects
+				(font
+					(size 1.27 1.27)
+				)
+			)
+		)
+		(property "Value" "Charger"
+			(at 147.32 132.08 90)
+			(show_name no)
+			(do_not_autoplace no)
+			(effects
+				(font
+					(size 1.27 1.27)
+				)
+			)
+		)
+		(property "Footprint" ""
+			(at 148.59 127 0)
+			(hide yes)
+			(show_name no)
+			(do_not_autoplace no)
+			(effects
+				(font
+					(size 1.27 1.27)
+				)
+			)
+		)
+		(property "Datasheet" ""
+			(at 148.59 127 0)
+			(hide yes)
+			(show_name no)
+			(do_not_autoplace no)
+			(effects
+				(font
+					(size 1.27 1.27)
+				)
+			)
+		)
+		(property "Description" "Generic connector, single row, 01x06, script generated"
+			(at 148.59 127 0)
+			(hide yes)
+			(show_name no)
+			(do_not_autoplace no)
+			(effects
+				(font
+					(size 1.27 1.27)
+				)
+			)
+		)
+		(pin "2"
+		)
+		(pin "6"
+		)
+		(pin "1"
+		)
+		(pin "5"
+		)
+		(pin "3"
+		)
+		(pin "4"
+		)
+		(instances
+			(project "Charger Junction PCB V1.01"
+				(path "/75f6fa4d-fba8-4d29-9299-863888d8bb95/37a81acb-7a57-4259-903f-870230a418d1/a56e1ce8-18bc-4320-87c8-0a13c817c3cf"
+					(reference "J6")
+					(unit 1)
+				)
+			)
+		)
+	)
+	(symbol
 		(lib_id "Connector:Conn_01x02_Socket")
-		(at 137.16 127 270)
-		(unit 1)
-		(body_style 1)
-		(exclude_from_sim no)
-		(in_bom yes)
-		(on_board yes)
-		(in_pos_files yes)
-		(dnp no)
-		(fields_autoplaced yes)
+		(at 114.3 127 270)
+		(unit 1)
+		(body_style 1)
+		(exclude_from_sim no)
+		(in_bom yes)
+		(on_board yes)
+		(in_pos_files yes)
+		(dnp no)
 		(property "Reference" "J3"
-			(at 138.43 125.0949 90)
-			(show_name no)
-			(do_not_autoplace no)
-			(effects
-				(font
-					(size 1.27 1.27)
-				)
-				(justify left)
-			)
-		)
-		(property "Value" "Charger CAN"
-			(at 138.43 127.6349 90)
+			(at 115.57 125.0949 90)
+			(show_name no)
+			(do_not_autoplace no)
+			(effects
+				(font
+					(size 1.27 1.27)
+				)
+				(justify left)
+			)
+		)
+		(property "Value" "J1772 In"
+			(at 108.712 129.794 90)
 			(show_name no)
 			(do_not_autoplace no)
@@
 		)
 		(property "Footprint" ""
-			(at 137.16 127 0)
+			(at 114.3 127 0)
 			(hide yes)
 			(show_name no)
@@
 		)
 		(property "Datasheet" ""
-			(at 137.16 127 0)
+			(at 114.3 127 0)
 			(hide yes)
 			(show_name no)
@@
 		)
 		(property "Description" "Generic connector, single row, 01x02, script generated"
-			(at 137.16 127 0)
+			(at 114.3 127 0)
 			(hide yes)
 			(show_name no)
@@
 		)
 		(instances
-			(project "Charger Master"
+			(project "Charger Junction PCB V1.01"
 				(path "/75f6fa4d-fba8-4d29-9299-863888d8bb95/37a81acb-7a57-4259-903f-870230a418d1/a56e1ce8-18bc-4320-87c8-0a13c817c3cf"
 					(reference "J3")
@@
 		)
 		(instances
-			(project "Charger Master"
+			(project "Charger Junction PCB V1.01"
 				(path "/75f6fa4d-fba8-4d29-9299-863888d8bb95/37a81acb-7a57-4259-903f-870230a418d1/a56e1ce8-18bc-4320-87c8-0a13c817c3cf"
 					(reference "R2")
@@
 		(in_pos_files yes)
 		(dnp no)
-		(fields_autoplaced yes)
 		(property "Reference" "D1"
-			(at 101.6 90.1699 90)
+			(at 93.472 89.408 90)
 			(show_name no)
 			(do_not_autoplace no)
@@
 			)
 		)
-		(property "Value" "SMAJ12CA"
-			(at 101.6 92.7099 90)
+		(property "Value" "Comchip ATV02W120B-HF"
+			(at 70.612 92.456 90)
 			(show_name no)
 			(do_not_autoplace no)
@@
 		)
 		(instances
-			(project "Charger Master"
+			(project "Charger Junction PCB V1.01"
 				(path "/75f6fa4d-fba8-4d29-9299-863888d8bb95/37a81acb-7a57-4259-903f-870230a418d1/a56e1ce8-18bc-4320-87c8-0a13c817c3cf"
 					(reference "D1")
@@
 		)
 		(instances
-			(project "Charger Master"
+			(project "Charger Junction PCB V1.01"
 				(path "/75f6fa4d-fba8-4d29-9299-863888d8bb95/37a81acb-7a57-4259-903f-870230a418d1/a56e1ce8-18bc-4320-87c8-0a13c817c3cf"
 					(reference "J5")
@@
 		)
 		(instances
-			(project "Charger Master"
+			(project "Charger Junction PCB V1.01"
 				(path "/75f6fa4d-fba8-4d29-9299-863888d8bb95/37a81acb-7a57-4259-903f-870230a418d1/a56e1ce8-18bc-4320-87c8-0a13c817c3cf"
 					(reference "#PWR04")
@@
 			)
 		)
-		(property "Footprint" "Diode_THT:D_DO-35_SOD27_P7.62mm_Horizontal"
+		(property "Footprint" "Diode_SMD:D_SOD-123"
 			(at 110.49 85.09 0)
 			(hide yes)
@@
 		)
 		(instances
-			(project "Charger Master"
+			(project "Charger Junction PCB V1.01"
 				(path "/75f6fa4d-fba8-4d29-9299-863888d8bb95/37a81acb-7a57-4259-903f-870230a418d1/a56e1ce8-18bc-4320-87c8-0a13c817c3cf"
 					(reference "D2")
@@
 		)
 		(instances
-			(project "Charger Master"
+			(project "Charger Junction PCB V1.01"
 				(path "/75f6fa4d-fba8-4d29-9299-863888d8bb95/37a81acb-7a57-4259-903f-870230a418d1/a56e1ce8-18bc-4320-87c8-0a13c817c3cf"
 					(reference "SW1")
