File: Charger/Charger Junction PCB V1.01/Charger Junction PCB V1.01.kicad_sch (KiCad schematic)
At the start: 26 parts, among them J1 3557-2, J10 BMS and IMD Indicator Light C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, J2 12V Battery, J3 Charger, J4 J1772 Plug, J5 3557-2, J6 Power Switch Connector, J7 E-Stop, J9 Reset Button, K1 Panasonic_TX2, K2 Panasonic_TX2, Q1 2N7002, Q2 2N7002, SW1 J1772 Dummy Enable (BMS Overr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

Commit message: Added diode bypass jumper
Parts:
- added JP?: Diode Bypass Jumper, symbol Jumper:Jumper_2_Bridged
Connections:
- net at D4.1, D4.2, J1.3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: now also JP?.2 (B)
- net at D4.3, J6.2 (Pin_2): now also JP?.1 (A)
Other:
- moved on the sheet: D4
Changed lines of the file:
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@@
 	)
 	(junction
-		(at 123.19 124.46)
+		(at 62.23 55.88)
 		(diameter 0)
 		(color 0 0 0 0)
 	)
 	(junction
-		(at 97.79 80.01)
+		(at 123.19 124.46)
 		(diameter 0)
 		(color 0 0 0 0)
 	)
 	(junction
-		(at 62.23 69.85)
+		(at 95.25 55.88)
 		(diameter 0)
 		(color 0 0 0 0)
 	)
 	(junction
-		(at 97.79 171.45)
+		(at 97.79 80.01)
 		(diameter 0)
 		(color 0 0 0 0)
 	)
 	(junction
-		(at 76.2 69.85)
+		(at 97.79 171.45)
 		(diameter 0)
 		(color 0 0 0 0)
 	)
 	(junction
-		(at 62.23 55.88)
+		(at 76.2 69.85)
 		(diameter 0)
 		(color 0 0 0 0)
@@
 	)
 	(junction
+		(at 63.5 43.18)
+		(diameter 0)
+		(color 0 0 0 0)
+	)
+	(junction
 		(at 137.16 30.48)
 		(diameter 0)
@@
 	)
 	(junction
+		(at 62.23 69.85)
+		(diameter 0)
+		(color 0 0 0 0)
+	)
+	(junction
 		(at 163.83 105.41)
 		(diameter 0)
@@
 	(wire
 		(pts
+			(xy 95.25 55.88) (xy 95.25 45.72)
+		)
+		(stroke
+			(width 0)
+			(type default)
+		)
+	)
+	(wire
+		(pts
 			(xy 147.32 106.68) (xy 147.32 107.95)
 		)
@@
 	(wire
 		(pts
-			(xy 132.08 102.87) (xy 114.3 102.87)
+			(xy 62.23 69.85) (xy 62.23 55.88)
 		)
 		(stroke
@@
 	(wire
 		(pts
-			(xy 119.38 100.33) (xy 115.57 100.33)
+			(xy 132.08 102.87) (xy 114.3 102.87)
 		)
 		(stroke
@@
 	(wire
 		(pts
-			(xy 77.47 77.47) (xy 77.47 101.6)
+			(xy 119.38 100.33) (xy 115.57 100.33)
 		)
 		(stroke
@@
 	(wire
 		(pts
-			(xy 158.75 102.87) (xy 158.75 80.01)
+			(xy 77.47 77.47) (xy 77.47 101.6)
 		)
 		(stroke
@@
 	(wire
 		(pts
-			(xy 76.2 69.85) (xy 76.2 72.39)
+			(xy 158.75 102.87) (xy 158.75 80.01)
 		)
 		(stroke
@@
 	(wire
 		(pts
-			(xy 26.67 156.21) (xy 41.91 156.21)
+			(xy 76.2 69.85) (xy 76.2 72.39)
 		)
 		(stroke
@@
 	(wire
 		(pts
-			(xy 62.23 53.34) (xy 62.23 55.88)
+			(xy 26.67 156.21) (xy 41.91 156.21)
 		)
 		(stroke
@@
 	(wire
 		(pts
-			(xy 62.23 55.88) (xy 62.23 69.85)
-		)
-		(stroke
-			(width 0)
-			(type default)
-		)
-	)
-	(wire
-		(pts
 			(xy 115.57 95.25) (xy 115.57 100.33)
 		)
@@
 	(wire
 		(pts
+			(xy 95.25 45.72) (xy 93.98 45.72)
+		)
+		(stroke
+			(width 0)
+			(type default)
+		)
+	)
+	(wire
+		(pts
 			(xy 207.01 128.27) (xy 210.82 128.27)
 		)
@@
 	(wire
 		(pts
+			(xy 62.23 43.18) (xy 63.5 43.18)
+		)
+		(stroke
+			(width 0)
+			(type default)
+		)
+	)
+	(wire
+		(pts
 			(xy 121.92 104.14) (xy 121.92 107.95)
 		)
@@
 	(wire
 		(pts
+			(xy 63.5 43.18) (xy 63.5 45.72)
+		)
+		(stroke
+			(width 0)
+			(type default)
+		)
+	)
+	(wire
+		(pts
 			(xy 210.82 128.27) (xy 210.82 130.81)
 		)
@@
 	(wire
 		(pts
-			(xy 95.25 55.88) (xy 92.71 55.88)
+			(xy 139.7 101.6) (xy 139.7 106.68)
 		)
 		(stroke
@@
 	(wire
 		(pts
-			(xy 139.7 101.6) (xy 139.7 106.68)
+			(xy 77.47 77.47) (xy 76.2 77.47)
 		)
 		(stroke
@@
 	(wire
 		(pts
-			(xy 77.47 77.47) (xy 76.2 77.47)
+			(xy 134.62 104.14) (xy 134.62 107.95)
 		)
 		(stroke
@@
 	(wire
 		(pts
-			(xy 134.62 104.14) (xy 134.62 107.95)
+			(xy 142.24 90.17) (xy 142.24 101.6)
 		)
 		(stroke
@@
 	(wire
 		(pts
-			(xy 142.24 90.17) (xy 142.24 101.6)
+			(xy 80.01 97.79) (xy 80.01 101.6)
 		)
 		(stroke
@@
 	(wire
 		(pts
-			(xy 80.01 97.79) (xy 80.01 101.6)
+			(xy 82.55 55.88) (xy 95.25 55.88)
 		)
 		(stroke
@@
 	(wire
 		(pts
+			(xy 62.23 55.88) (xy 62.23 43.18)
+		)
+		(stroke
+			(width 0)
+			(type default)
+		)
+	)
+	(wire
+		(pts
 			(xy 177.8 102.87) (xy 177.8 80.01)
 		)
@@
 	(wire
 		(pts
+			(xy 62.23 55.88) (xy 72.39 55.88)
+		)
+		(stroke
+			(width 0)
+			(type default)
+		)
+	)
+	(wire
+		(pts
 			(xy 214.63 129.54) (xy 214.63 133.35)
 		)
@@
 	(symbol
 		(lib_id "PMEG045V100EPE-QZ:PMEG100V080ELPDZ")
-		(at 62.23 53.34 0)
+		(at 63.5 43.18 0)
 		(unit 1)
 		(body_style 1)
@@
 		(dnp no)
 		(property "Reference" "D4"
-			(at 77.47 46.99 0)
+			(at 78.74 36.83 0)
 			(show_name no)
 			(do_not_autoplace no)
@@
 		)
 		(property "Value" "PMEG045V100EPE-QZ"
-			(at 77.47 49.784 0)
+			(at 78.74 39.624 0)
 			(show_name no)
 			(do_not_autoplace no)
@@
 		)
 		(property "Footprint" "Charger PCB:SOT1289_CFP15_NEX"
-			(at 62.23 53.34 0)
+			(at 63.5 43.18 0)
 			(hide yes)
 			(show_name no)
@@
 		)
 		(property "Datasheet" "https://assets.nexperia.com/documents/data-sheet/PMEG045V100EPE-Q.pdf"
-			(at 62.23 53.34 0)
+			(at 63.5 43.18 0)
 			(hide yes)
 			(show_name no)
@@
 		)
 		(property "Description" ""
-			(at 62.23 53.34 0)
+			(at 63.5 43.18 0)
 			(hide yes)
 			(show_name no)
@@
 					(unit 1)
 				)
+			)
+		)
+	)
+	(symbol
+		(lib_id "Jumper:Jumper_2_Bridged")
+		(at 77.47 55.88 180)
+		(unit 1)
+		(body_style 1)
+		(exclude_from_sim no)
+		(in_bom yes)
+		(on_board yes)
+		(in_pos_files yes)
+		(dnp no)
+		(fields_autoplaced yes)
+		(property "Reference" "JP?"
+			(at 77.47 50.8 0)
+			(show_name no)
+			(do_not_autoplace no)
+			(effects
+				(font
+					(size 1.27 1.27)
+				)
+			)
+		)
+		(property "Value" "Diode Bypass Jumper"
+			(at 77.47 53.34 0)
+			(show_name no)
+			(do_not_autoplace no)
+			(effects
+				(font
+					(size 1.27 1.27)
+				)
+			)
+		)
+		(property "Footprint" ""
+			(at 77.47 55.88 0)
+			(hide yes)
+			(show_name no)
+			(do_not_autoplace no)
+			(effects
+				(font
+					(size 1.27 1.27)
+				)
+			)
+		)
+		(property "Datasheet" ""
+			(at 77.47 50.8 0)
+			(hide yes)
+			(show_name no)
+			(do_not_autoplace no)
+			(effects
+				(font
+					(size 1.27 1.27)
+				)
+			)
+		)
+		(property "Description" "Jumper, 2-pole, closed/bridged"
+			(at 77.47 48.26 0)
+			(hide yes)
+			(show_name no)
+			(do_not_autoplace no)
+			(effects
+				(font
+					(size 1.27 1.27)
+				)
+			)
+		)
+		(pin "2"
+		)
+		(pin "1"
+		)
+		(instances
+			(project "Charger Junction PCB V1.01"
+				(path "/75f6fa4d-fba8-4d29-9299-863888d8bb95"
+					(reference "JP?")
+					(unit 1)
+				)
